File: arduino_icsp_shield/arduino_icsp_shield.kicad_sch (KiCad schematic)
At the start: 18 parts, among them J1 Power, J2 Digital/PWM, J3 Analog, J4 Digital/PWM, J5 ICSP, SW1 TARGET RESET, U1 ADG3304

Commit message: Fix which voltage the level shifter enable is coming from
Connections:
- net +5V: no longer R4.1
- net ICSP_VCC: now also R4.1
Other:
- note added: "EN signal should be referenced to VCCA"
Changed lines of the file:
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@@
     (stroke (width 0) (type solid))
   )
-  (wire (pts (xy 177.8 92.71) (xy 177.8 93.98))
+  (wire (pts (xy 187.96 91.44) (xy 177.8 91.44))
+    (stroke (width 0) (type default))
+  )
+  (wire (pts (xy 177.8 91.44) (xy 177.8 93.98))
     (stroke (width 0) (type default))
   )
@@
     (stroke (width 0) (type default))
   )
-  (text "VCCA must be less than\nor equal to VCCY" (at 151.13 114.3 0)
+  (text "VCCA must be less than\nor equal to VCCY" (at 106.68 109.22 0)
+    (effects (font (size 1.27 1.27)) (justify left bottom))
+  )
+  (text "EN signal should be\nreferenced to VCCA" (at 157.48 111.76 0)
     (effects (font (size 1.27 1.27)) (justify left bottom))
   )
@@
   )
   (label "D10{slash}RESET" (at 88.9 60.96 180) (fields_autoplaced)
+    (effects (font (size 1.27 1.27)) (justify right bottom))
+  )
+  (label "ICSP_VCC" (at 187.96 91.44 180) (fields_autoplaced)
     (effects (font (size 1.27 1.27)) (justify right bottom))
   )
@@
         )
       )
-    )
-  )
-  (symbol (lib_id "power:+5V") (at 177.8 92.71 0) (mirror y) (unit 1)
-    (in_bom yes) (on_board yes) (dnp no)
-    (property "Reference" "#PWR013" (at 177.8 96.52 0)
-      (effects (font (size 1.27 1.27)) hide)
-    )
-    (property "Value" "+5V" (at 177.8 88.9 0)
-      (effects (font (size 1.27 1.27)))
-    )
-    (property "Footprint" "" (at 177.8 92.71 0)
-      (effects (font (size 1.27 1.27)))
-    )
-    (property "Datasheet" "" (at 177.8 92.71 0)
-      (effects (font (size 1.27 1.27)))
-    )
-    (pin "1")
-    (instances
-      (project "arduino_icsp_shield"
-        (path "/e63e39d7-6ac0-4ffd-8aa3-1841a4541b55"
-          (reference "#PWR013") (unit 1)
-        )
-      )
