File: arduino_icsp_shield/arduino_icsp_shield.kicad_pcb (KiCad board)
At the start: 2 copper layers, 53.3 x 68.6 mm, 22 parts, among them J1 Power, J2 Digital/PWM, J3 Analog, J4 Digital/PWM, J5 ICSP, SW1 TARGET RESET, U1 ADG3304

Commit message: Fix which voltage the level shifter enable is coming from
Parts:
- moved R4 3.76 mm to (119.0, 79.0), turned to 90 degrees
Connections:
- R4 pad 1: +5V -> /ICSP_VCC
Changed lines of the file:
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@@
   )
   (footprint "Resistor_SMD:R_0805_2012Metric" (layer "F.Cu")
-    (at 119.05 75.2585 -90)
+    (at 119.05 79.0215 90)
     (descr "Resistor SMD 0805 (2012 Metric), square (rectangular) end terminal, IPC_7351 nominal, (Body size source: IPC-SM-782 page 72, https://www.pcb-3d.com/wordpress/wp-content/uploads/ipc-sm-782a_amendment_1_and_2.pdf), generated with kicad-footprint-generator")
     (tags "resistor")
@@
     (fp_line (start 1 0.625) (end -1 0.625)
       (stroke (width 0.1) (type solid)) (layer "F.Fab"))
-    (pad "1" smd roundrect (at -0.9125 0 270) (size 1.025 1.4) (layers "F.Cu" "F.Paste" "F.Mask") (roundrect_rratio 0.243902439)
-      (net 3 "+5V") (pintype "passive"))
-    (pad "2" smd roundrect (at 0.9125 0 270) (size 1.025 1.4) (layers "F.Cu" "F.Paste" "F.Mask") (roundrect_rratio 0.243902439)
+    (pad "1" smd roundrect (at -0.9125 0 90) (size 1.025 1.4) (layers "F.Cu" "F.Paste" "F.Mask") (roundrect_rratio 0.243902439)
+      (net 9 "/ICSP_VCC") (pintype "passive"))
+    (pad "2" smd roundrect (at 0.9125 0 90) (size 1.025 1.4) (layers "F.Cu" "F.Paste" "F.Mask") (roundrect_rratio 0.243902439)
       (net 39 "/ENABLE") (pintype "passive"))
     (model "${KICAD6_3DMODEL_DIR}/Resistor_SMD.3dshapes/R_0805_2012Metric.wrl"
@@
   (segment (start 127.48 91.57) (end 113.43 91.57) (width 0.4) (layer "F.Cu") (net 38))
   (segment (start 128.62 76) (end 128.62 74.2775) (width 0.4) (layer "F.Cu") (net 39))
-  (segment (start 119.05 76.171) (end 119.05 77.14) (width 0.4) (layer "F.Cu") (net 39))
+  (segment (start 119.05 78.109) (end 119.05 77.14) (width 0.4) (layer "F.Cu") (net 39))
   (via (at 119.05 77.14) (size 0.6) (drill 0.3) (layers "F.Cu" "B.Cu") (net 39))
   (via (at 128.62 76) (size 0.6) (drill 0.3) (layers "F.Cu" "B.Cu") (net 39))

Commit message: Tweak resistor placement
Parts:
- moved R4 0.51 mm to (119.6, 79.0)
Routing:
- net /ENABLE: track 12.7 -> 12.2 mm
- net GND: vias 70 -> 71
Changed lines of the file:
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@@
   )
   (footprint "Resistor_SMD:R_0805_2012Metric" (layer "F.Cu")
-    (at 119.05 79.0215 90)
+    (at 119.558 79.0215 90)
     (descr "Resistor SMD 0805 (2012 Metric), square (rectangular) end terminal, IPC_7351 nominal, (Body size source: IPC-SM-782 page 72, https://www.pcb-3d.com/wordpress/wp-content/uploads/ipc-sm-782a_amendment_1_and_2.pdf), generated with kicad-footprint-generator")
     (tags "resistor")
@@
   (via (at 121.59 99.365) (size 0.6) (drill 0.3) (layers "F.Cu" "B.Cu") (free) (net 1))
   (via (at 121.42 75.75) (size 0.6) (drill 0.3) (layers "F.Cu" "B.Cu") (free) (net 1))
+  (via (at 117.526 78.41) (size 0.6) (drill 0.3) (layers "F.Cu" "B.Cu") (free) (net 1))
   (via (at 130.48 88.57) (size 0.6) (drill 0.3) (layers "F.Cu" "B.Cu") (free) (net 1))
   (via (at 107.62 93.015) (size 0.6) (drill 0.3) (layers "F.Cu" "B.Cu") (free) (net 1))
@@
   (segment (start 129.21 89.84) (end 127.48 91.57) (width 0.4) (layer "F.Cu") (net 38))
   (segment (start 127.48 91.57) (end 113.43 91.57) (width 0.4) (layer "F.Cu") (net 38))
+  (segment (start 119.558 78.109) (end 119.558 77.14) (width 0.4) (layer "F.Cu") (net 39))
   (segment (start 128.62 76) (end 128.62 74.2775) (width 0.4) (layer "F.Cu") (net 39))
-  (segment (start 119.05 78.109) (end 119.05 77.14) (width 0.4) (layer "F.Cu") (net 39))
-  (via (at 119.05 77.14) (size 0.6) (drill 0.3) (layers "F.Cu" "B.Cu") (net 39))
+  (via (at 119.558 77.14) (size 0.6) (drill 0.3) (layers "F.Cu" "B.Cu") (net 39))
   (via (at 128.62 76) (size 0.6) (drill 0.3) (layers "F.Cu" "B.Cu") (net 39))
-  (segment (start 128.62 76) (end 127.48 77.14) (width 0.4) (layer "B.Cu") (net 39))
-  (segment (start 127.48 77.14) (end 119.05 77.14) (width 0.4) (layer "B.Cu") (net 39))
+  (segment (start 127.48 77.14) (end 128.62 76) (width 0.4) (layer "B.Cu") (net 39))
+  (segment (start 119.558 77.14) (end 127.48 77.14) (width 0.4) (layer "B.Cu") (net 39))
   (segment (start 125.37 80.799878) (end 120.599878 85.57) (width 0.4) (layer "F.Cu") (net 42))
   (segment (start 125.37 80.0025) (end 125.37 80.799878) (width 0.4) (layer "F.Cu") (net 42))
